Commit message: added jamal xacro

File: legged_examples/legged_unitree/legged_unitree_description/urdf/common/leg.xacro (robot description, xacro)
@@ -108,5 +108,5 @@
         <link name="${prefix}_calf">
             <visual>
-                <origin rpy="0 0 0" xyz="0 0 0"/>
+                <origin rpy="0 0.06 0" xyz="0 0 0"/>
                 <geometry>
                     <mesh filename="${mesh_path}/calf.dae"

File: legged_examples/legged_unitree/legged_unitree_description/urdf/robot.xacro (robot description, xacro)
@@ -1,5 +1,5 @@
 <?xml version="1.0"?>
 <robot xmlns:xacro="http://www.ros.org/wiki/xacro" name="robot">
-    <xacro:arg name="robot_type" default="a1"/>
+    <xacro:arg name="robot_type" default="jamal"/>
     <xacro:include filename="$(find legged_unitree_description)/urdf/common/materials.xacro"/>
     <xacro:include filename="$(find legged_unitree_description)/urdf/common/leg.xacro"/>

Commit message: hardware testing 14-8 1

File: legged_examples/legged_unitree/legged_unitree_description/urdf/common/leg.xacro (robot description, xacro)
@@ -33,5 +33,5 @@
                 </xacro:if>
                 <geometry>
-                    <mesh filename="${mesh_path}/hip.dae"
+                    <mesh filename="${mesh_path}/hip.STL"
                           scale="1 1 1"/>
                 </geometry>
@@ -67,9 +67,9 @@
                 <geometry>
                     <xacro:if value="${mirror_dae == True}">
-                        <mesh filename="${mesh_path}/thigh.dae"
+                        <mesh filename="${mesh_path}/thigh.STL"
                               scale="1 1 1"/>
                     </xacro:if>
                     <xacro:if value="${mirror_dae == False}">
-                        <mesh filename="${mesh_path}/thigh_mirror.dae"
+                        <mesh filename="${mesh_path}/thigh_mirror.STL"
                               scale="1 1 1"/>
                     </xacro:if>
@@ -110,5 +110,5 @@
                 <origin rpy="0 0.06 0" xyz="0 0 0"/>
                 <geometry>
-                    <mesh filename="${mesh_path}/calf.dae"
+                    <mesh filename="${mesh_path}/calf.STL"
                           scale="1 1 1"/>
                 </geometry>

File: legged_examples/legged_unitree/legged_unitree_description/urdf/robot.xacro (robot description, xacro)
@@ -13,5 +13,5 @@
             <origin rpy="0 0 0" xyz="0 0 0"/>
             <geometry>
-                <mesh filename="${mesh_path}/trunk.dae" scale="1 1 1"/>
+                <mesh filename="${mesh_path}/trunk.STL" scale="1 1 1"/>
             </geometry>
         </visual>

Commit message: solved rviz robot visualization

File: legged_examples/legged_unitree/legged_unitree_description/urdf/common/leg.xacro (robot description, xacro)
@@ -33,5 +33,5 @@
                 </xacro:if>
                 <geometry>
-                    <mesh filename="${mesh_path}/hip.STL"
+                    <mesh filename="${mesh_path}/hip.dae"
                           scale="1 1 1"/>
                 </geometry>
@@ -67,9 +67,9 @@
                 <geometry>
                     <xacro:if value="${mirror_dae == True}">
-                        <mesh filename="${mesh_path}/thigh.STL"
+                        <mesh filename="${mesh_path}/thigh.dae"
                               scale="1 1 1"/>
                     </xacro:if>
                     <xacro:if value="${mirror_dae == False}">
-                        <mesh filename="${mesh_path}/thigh_mirror.STL"
+                        <mesh filename="${mesh_path}/thigh_mirror.dae"
                               scale="1 1 1"/>
                     </xacro:if>
@@ -110,5 +110,5 @@
                 <origin rpy="0 0.06 0" xyz="0 0 0"/>
                 <geometry>
-                    <mesh filename="${mesh_path}/calf.STL"
+                    <mesh filename="${mesh_path}/calf.dae"
                           scale="1 1 1"/>
                 </geometry>

File: legged_examples/legged_unitree/legged_unitree_description/urdf/robot.xacro (robot description, xacro)
@@ -8,10 +8,10 @@
     <xacro:include filename="$(find legged_unitree_description)/urdf/$(arg robot_type)/const.xacro"/>
 <!--    <xacro:property name="mesh_path" value="../meshes"/>-->
-    <xacro:property name="mesh_path" value="$(find legged_unitree_description)/meshes/$(arg robot_type)"/>
+    <xacro:property name="mesh_path" value="file://$(find legged_unitree_description)/meshes/$(arg robot_type)"/>
     <link name="base">
         <visual>
             <origin rpy="0 0 0" xyz="0 0 0"/>
             <geometry>
-                <mesh filename="${mesh_path}/trunk.STL" scale="1 1 1"/>
+                <mesh filename="${mesh_path}/trunk.dae" scale="1 1 1"/>
             </geometry>
         </visual>
