Commit message: hardware testing 19-8 4

File: legged_examples/legged_unitree/legged_unitree_description/urdf/jamal/const.xacro (robot description, xacro)
@@ -65,6 +65,6 @@
     <!-- trunk -->
     <xacro:property name="trunk_mass" value="13.2256112448737"/>
-    <xacro:property name="trunk_com_x" value="0.0"/>
-    <xacro:property name="trunk_com_y" value="0.002"/>
+    <xacro:property name="trunk_com_x" value="-0.025"/>
+    <xacro:property name="trunk_com_y" value="0"/>
     <xacro:property name="trunk_com_z" value="-0.0005"/>
     <xacro:property name="trunk_ixx" value="0.0574649406584405"/>
